File: Master Design Reference/USB-C_Power_Supply/USB-C_Power_Supply.kicad_sch (KiCad schematic)
At the start: 51 parts, among them J1 691137710002, J10 Conn_01x04_Pin, J11 Conn_01x04_Pin, J12 Conn_01x03_Pin, J13 Conn_01x03_Pin, J14 Conn_01x03_Pin, J15 Conn_01x03_Pin, J16 691137710002, J2 691137710002, J4 691137710002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

Commit message: Week02 Resources
Parts:
- removed U1, U2: LM2596S-ADJ, Package_TO_SOT_SMD:TO-263-5_TabPin3, symbol Regulator_Switching:LM2596S-ADJ
- added U1, U2: LM2576T-ADJ, Package_TO_SOT_THT:TO-220-5_Vertical, symbol Regulator_Switching:LM2576T-ADJ
- C1, C8: footprint (none) -> Capacitor_THT:CP_Radial_D8.0mm_P3.50mm
- C2: renamed from C5; footprint (none) -> Capacitor_THT:CP_Radial_D8.0mm_P3.50mm
- C3: renamed from C2; footprint (none) -> Capacitor_SMD:C_0805_2012Metric
- C4: renamed from C6; footprint (none) -> Capacitor_SMD:C_0805_2012Metric
- C5: renamed from C3; footprint (none) -> Capacitor_THT:CP_Radial_D8.0mm_P3.50mm
- C6: renamed from C7; footprint (none) -> Capacitor_THT:CP_Radial_D8.0mm_P3.50mm
- C7: renamed from C4; footprint (none) -> Capacitor_THT:CP_Radial_D8.0mm_P3.50mm
- D1: renamed from D7; footprint (none) -> LED_SMD:LED_0805_2012Metric
- D2: renamed from D6; footprint (none) -> LED_SMD:LED_0805_2012Metric
- D3: renamed from D1; footprint (none) -> Diode_SMD:D_SMA
- D4: renamed from D3; footprint (none) -> Diode_SMD:D_SMA
- D5: renamed from D2; footprint (none) -> LED_SMD:LED_0805_2012Metric
- D6: renamed from D5; footprint (none) -> LED_SMD:LED_0805_2012Metric
- HS1, HS2: footprint 63710ABPE -> USB-C Supply:63710ABPE
- J1: renamed from J4; footprint (none) -> TerminalBlock_Phoenix:TerminalBlock_Phoenix_MKDS-1,5-2_1x02_P5.00mm_Horizontal
- J10: renamed from J12; footprint (none) -> Connector_PinHeader_2.54mm:PinHeader_1x03_P2.54mm_Vertical
- J11: renamed from J13; footprint (none) -> Connector_PinHeader_2.54mm:PinHeader_1x03_P2.54mm_Vertical
- J12: renamed from J16; footprint (none) -> TerminalBlock_Phoenix:TerminalBlock_Phoenix_MKDS-1,5-2_1x02_P5.00mm_Horizontal
- J13: renamed from J14; footprint (none) -> Connector_PinHeader_2.54mm:PinHeader_1x03_P2.54mm_Vertical
- J14: renamed from J15; footprint (none) -> Connector_PinHeader_2.54mm:PinHeader_1x03_P2.54mm_Vertical
- J15: renamed from J2; footprint (none) -> TerminalBlock_Phoenix:TerminalBlock_Phoenix_MKDS-1,5-2_1x02_P5.00mm_Horizontal
- J2: renamed from J1; footprint (none) -> TerminalBlock_Phoenix:TerminalBlock_Phoenix_MKDS-1,5-2_1x02_P5.00mm_Horizontal
- J3: renamed from J7; footprint (none) -> Connector_BarrelJack:BarrelJack_CUI_PJ-063AH_Horizontal
- J4: renamed from J5; footprint (none) -> Connector_PinHeader_2.54mm:PinHeader_1x02_P2.54mm_Vertical
- J5: renamed from J6; footprint (none) -> Connector_PinHeader_2.54mm:PinHeader_1x02_P2.54mm_Vertical
- J6: renamed from J8; footprint (none) -> Connector_PinHeader_2.54mm:PinHeader_1x04_P2.54mm_Vertical
- J7: renamed from J9; footprint (none) -> Connector_PinHeader_2.54mm:PinHeader_1x04_P2.54mm_Vertical
- J8: renamed from J10; footprint (none) -> Connector_PinHeader_2.54mm:PinHeader_1x04_P2.54mm_Vertical
- J9: renamed from J11; footprint (none) -> Connector_PinHeader_2.54mm:PinHeader_1x04_P2.54mm_Vertical
- L1: footprint (none) -> Inductor_SMD:L_Bourns_SRR1210A
- L2: renamed from L3; footprint (none) -> Inductor_SMD:L_Bourns_SRR1210A
- L3: renamed from L2; footprint (none) -> Inductor_SMD:L_APV_ANR5020
- L4: footprint (none) -> Inductor_SMD:L_APV_ANR5020
- M1: footprint USB_C-PD -> USB-C Supply:USB_C-PD
- R1, R8: footprint (none) -> Resistor_SMD:R_0805_2012Metric
- R10: renamed from R5; footprint (none) -> Resistor_SMD:R_0805_2012Metric
- R2: renamed from R3; footprint (none) -> Resistor_SMD:R_0805_2012Metric
- R3: renamed from R11; footprint (none) -> Resistor_SMD:R_0805_2012Metric
- R4: renamed from R9; footprint (none) -> Resistor_SMD:R_0805_2012Metric
- R5: renamed from R12; footprint (none) -> Resistor_SMD:R_0805_2012Metric
- R6: renamed from R10; footprint (none) -> Resistor_SMD:R_0805_2012Metric
- R7: renamed from R6; footprint (none) -> Resistor_SMD:R_0805_2012Metric
- R9: renamed from R4; footprint (none) -> Resistor_SMD:R_0805_2012Metric
- RV1, RV2: footprint (none) -> Potentiometer_THT:Potentiometer_Vishay_T73YP_Vertical
- SW1: renamed from SW2; footprint (none) -> USB-C Supply:GF1260305
Connections:
- net GND_A: now also U1.3 (GND), U1.5 (~{ON}/OFF)
- net GND_B: now also U2.3 (GND), U2.5 (~{ON}/OFF)
- net V_IN_A: now also U1.1 (VIN)
- net V_IN_B: now also U2.1 (VIN)
- net at R4.2, RV2.2, RV2.3: now also U2.4 (FB)
- net at R3.2, RV1.2, RV1.3: now also U1.4 (FB)
- net at D3.1 (K), L1.1: now also U1.2 (OUT)
- net at D4.1 (K), L2.1: now also U2.2 (OUT)
